Commit message: Finished visual design

File: mecabot_body/urdf/mecabot_core.xacro (robot description, xacro)
@@ -4,4 +4,7 @@
     <xacro:property name="layer_w" value="0.15"/>
     <xacro:property name="layer_h" value="0.002"/>
+    <xacro:property name="chassis_l" value="${layer_l}"/>
+    <xacro:property name="chassis_w" value="${layer_w}"/>
+    <xacro:property name="chassis_h" value="0.07"/>
     <xacro:property name="PI" value="3.1415926535897931" />
     <xacro:property name="wheel_radius" value="0.03" />
@@ -14,7 +17,7 @@
     <link name="base_link">
         <collision>
-            <origin xyz="0.0 0.0 ${0.07/2}" rpy="0.0 0.0 0.0"/>
+            <origin xyz="0.0 0.0 ${chassis_h/2}" rpy="0.0 0.0 0.0"/>
             <geometry>
-                <box size="${layer_l} ${layer_w} 0.07"/>
+                <box size="${chassis_l} ${chassis_w} ${chassis_h}"/>
             </geometry>
         </collision>

File: mecabot_body/urdf/parts/layer.xacro (robot description, xacro)
@@ -1,7 +1,19 @@
 <?xml version="1.0"?>
 <robot xmlns:xacro="http://www.ros.org/wiki/xacro">
-    <xacro:property name="side_piece_size" value="0.032"/>
+    <xacro:property name="side_piece_size" value="0.02"/>
+    <xacro:property name="motor_l" value = "0.07"/>
+    <xacro:property name="motor_w" value = "0.022"/>
+    <xacro:property name="motor_h" value = "0.018"/>
+    <xacro:property name="motor_offset_fb" value = "0.04"/>
+    <xacro:property name="motor_offset_lr" value = "0.034"/>
     <xacro:macro name="base_color">
-        <color rgba="0.20 0.20 0.20 1.0"/>
+        <material name="metal">
+            <color rgba="0.5 0.5 0.5 1.0"/>
+        </material>
+    </xacro:macro>
+    <xacro:macro name="motor_color">
+        <material name="motor">
+            <color rgba="${247/255} ${200/255} ${60/255} 1.0"/>
+        </material>
     </xacro:macro>
     <xacro:macro name="layer" params="prefix parent length width height reflect">
@@ -14,4 +26,45 @@
                 <xacro:base_color/>
             </visual>
+            <xacro:if value="${prefix == 'upper'}">
+                <visual name="direction_piece">
+                    <origin xyz="${length/2-side_piece_size/2} 0.0 ${height/2}" rpy="0.0 0.0 0.0"/>
+                    <geometry>
+                        <box size="${side_piece_size} ${side_piece_size} ${height}"/>
+                    </geometry>
+                    <material name="header">
+                        <color rgba="1.0 0.0 0.0 1.0"/>
+                    </material>
+                </visual>
+            </xacro:if>
+            <xacro:if value="${prefix == 'lower'}">
+                <visual name="FL_motor">
+                    <origin xyz="${motor_offset_fb} ${motor_offset_lr} -${motor_h/2}" rpy="0.0 0.0 0.0"/>
+                    <geometry>
+                        <box size="${motor_l} ${motor_w} ${motor_h}"/>
+                    </geometry>
+                    <xacro:motor_color/>
+                </visual>
+                <visual name="FR_motor">
+                    <origin xyz="${motor_offset_fb} -${motor_offset_lr} -${motor_h/2}" rpy="0.0 0.0 0.0"/>
+                    <geometry>
+                        <box size="${motor_l} ${motor_w} ${motor_h}"/>
+                    </geometry>
+                    <xacro:motor_color/>
+                </visual>
+                <visual name="BL_motor">
+                    <origin xyz="-${motor_offset_fb} ${motor_offset_lr} -${motor_h/2}" rpy="0.0 0.0 0.0"/>
+                    <geometry>
+                        <box size="${motor_l} ${motor_w} ${motor_h}"/>
+                    </geometry>
+                    <xacro:motor_color/>
+                </visual>
+                <visual name="BR_motor">
+                    <origin xyz="-${motor_offset_fb} -${motor_offset_lr} -${motor_h/2}" rpy="0.0 0.0 0.0"/>
+                    <geometry>
+                        <box size="${motor_l} ${motor_w} ${motor_h}"/>
+                    </geometry>
+                    <xacro:motor_color/>
+                </visual>
+            </xacro:if>
             <visual name="${prefix}_top_left_piece">
                 <origin xyz="${length/2-side_piece_size/2} ${width/2+side_piece_size/2} 0" rpy="0.0 0.0 0.0"/>
@@ -56,9 +109,15 @@
                 <xacro:base_color/>
             </visual>
+            <collision>
+                <origin xyz="0 0 0" rpy="0 0 0"/>
+                <geometry>
+                    <box size="${length} ${width + 2*side_piece_size} ${height}"/>
+                </geometry>
+            </collision>
         </link>
         <joint name="${parent}_to_${prefix}_layer_joint" type="fixed">
             <parent link="${parent}_link"/>
             <child link="${prefix}_layer_link"/>
-            <origin xyz="0 0 ${reflect*0.065}" rpy="0 0 0"/>
+            <origin xyz="0 0 ${reflect*0.055}" rpy="0 0 0"/>
         </joint>
     </xacro:macro>

File: mecabot_body/urdf/parts/pillar.xacro (robot description, xacro)
@@ -2,8 +2,8 @@
 <robot xmlns:xacro="http://ros.org/wiki/xacro">
     <xacro:property name="pillar_radius" value="0.002"/>
-    <xacro:property name="pillar_length" value="0.065"/>
+    <xacro:property name="pillar_length" value="0.055"/>
     <xacro:property name="pillar_mass" value="0.01"/>
-    <xacro:property name="pillar_offset_fb" value="0.11"/>
-    <xacro:property name="pillar_offset_lr" value="0.06"/>
+    <xacro:property name="pillar_offset_fb" value="0.12"/>
+    <xacro:property name="pillar_offset_lr" value="0.055"/>
     <xacro:macro name="pillar" params="suffix parent side_FB side_LR">
         <xacro:macro name="pillar_joint_origin">
@@ -18,6 +18,12 @@
                 <material name="pillar_color">
                     <color rgba="${255/255} ${108/255} ${12/255} 1.0"/>
-                  </material>
+                </material>
             </visual>
+            <collision>
+                <origin xyz="0.0 0.0 ${pillar_length/2}" rpy="0.0 0.0 0.0"/>
+                <geometry>
+                    <cylinder radius="${pillar_radius}" length="${pillar_length}"/>
+                </geometry>
+            </collision>
         </link>
         <joint name="${parent}_to_pillar_${suffix}_joint" type="fixed">

File: mecabot_body/urdf/wheels/wheel.xacro (robot description, xacro)
@@ -1,5 +1,5 @@
 <?xml version="1.0"?>
 <robot xmlns:xacro="http://www.ros.org/wiki/xacro">
-    <xacro:property name="motor_offset_z" value="0.012" />
+    <xacro:property name="motor_offset_z" value="0.009" />
     <xacro:property name="PI" value="3.1415926535897931" />
     <xacro:property name="wheel_radius" value="0.03" />
@@ -7,5 +7,5 @@
     <xacro:property name="wheel_mass" value="0.1" /> <!-- in kg-->
     <xacro:property name="wheel_offset_fb" value="0.06215"/>
-    <xacro:property name="wheel_offset_lr" value="0.062"/>
+    <xacro:property name="wheel_offset_lr" value="0.064"/>
     <xacro:macro name="cylinder_inertia" params="m r h">
         <inertia  ixx="${m*(3*r*r+h*h)/12}" ixy = "0" ixz = "0"
@@ -18,4 +18,13 @@
         </xacro:macro>
         <link name="${prefix}_wheel_link">
+            <visual name="shaft">
+                <origin xyz="0.0 0.0 ${-1 * side_LR * wheel_thickness/2}"/>
+                <geometry>
+                    <cylinder radius="0.0025" length="0.02"/>
+                </geometry>
+                <material name="white">
+                    <color rgba="1.0 1.0 1.0 1.0"/>
+                </material>
+            </visual>
             <visual>
                 <origin xyz="0.0 0.0 0.0" rpy="0.0 0.0 0.0"/>
@@ -24,5 +33,5 @@
                 </geometry>
                 <material name="yellow">
-                    <color rgba="${247/255} ${237/255} ${49/255} 1.0"/>
+                    <color rgba="${255/255} ${237/255} ${40/255} 1.0"/>
                 </material>
             </visual>
