Commit message: Added physical properties

File: mecabot_body/urdf/chassis/layer.xacro (robot description, xacro)
@@ -1,10 +1,11 @@
 <?xml version="1.0"?>
 <robot xmlns:xacro="http://www.ros.org/wiki/xacro">
-    <xacro:property name="side_piece_size" value="0.02"/>
-    <xacro:property name="motor_l" value = "0.07"/>
-    <xacro:property name="motor_w" value = "0.022"/>
-    <xacro:property name="motor_h" value = "0.018"/>
-    <xacro:property name="motor_offset_fb" value = "0.04"/>
-    <xacro:property name="motor_offset_lr" value = "0.034"/>
+    <xacro:property name="side_piece_size" value="0.03"/>
+    <xacro:property name="motor_l" value="0.07"/>
+    <xacro:property name="motor_w" value="0.022"/>
+    <xacro:property name="motor_h" value="0.018"/>
+    <xacro:property name="motor_offset_fb" value="0.04"/>
+    <xacro:property name="motor_offset_lr" value="0.034"/>
+    <xacro:property name="layer_mass" value="0.07"/>
     <xacro:macro name="base_color">
         <material name="metal">
@@ -17,5 +18,17 @@
         </material>
     </xacro:macro>
+    <xacro:macro name="inertial_box" params="mass x y z *origin">
+        <inertial>
+            <xacro:insert_block name="origin"/>
+            <mass value="${mass}" />
+            <inertia ixx="${(1/12) * mass * (y*y+z*z)}" ixy="0.0" ixz="0.0"
+                    iyy="${(1/12) * mass * (x*x+z*z)}" iyz="0.0"
+                    izz="${(1/12) * mass * (x*x+y*y)}" />
+        </inertial>
+    </xacro:macro>
     <xacro:macro name="layer" params="prefix parent length width height reflect">
+        <xacro:property name="layer_joint_origin">
+            <origin xyz="0 0 ${reflect*0.055}" rpy="0 0 0"/>
+        </xacro:property>
         <link name="${prefix}_layer_link">
             <visual>
@@ -27,6 +40,24 @@
             </visual>
             <xacro:if value="${prefix == 'upper'}">
-                <visual name="direction_piece">
+                <visual name="direction_piece_1">
                     <origin xyz="${length/2-side_piece_size/2} 0.0 ${height/2}" rpy="0.0 0.0 0.0"/>
+                    <geometry>
+                        <box size="${side_piece_size} ${side_piece_size} ${height/2}"/>
+                    </geometry>
+                    <material name="header">
+                        <color rgba="1.0 0.0 0.0 1.0"/>
+                    </material>
+                </visual>
+                <visual name="direction_piece_2">
+                    <origin xyz="${length/2-1.5*side_piece_size} ${width/2-side_piece_size/2} ${height/2}" rpy="0.0 0.0 0.0"/>
+                    <geometry>
+                        <box size="${side_piece_size} ${side_piece_size} ${height/2}"/>
+                    </geometry>
+                    <material name="header">
+                        <color rgba="1.0 0.0 0.0 1.0"/>
+                    </material>
+                </visual>
+                <visual name="direction_piece_3">
+                    <origin xyz="${length/2-1.5*side_piece_size} -${width/2-side_piece_size/2} ${height/2}" rpy="0.0 0.0 0.0"/>
                     <geometry>
                         <box size="${side_piece_size} ${side_piece_size} ${height}"/>
@@ -115,9 +146,12 @@
                 </geometry>
             </collision>
+            <xacro:inertial_box mass="${layer_mass}" x="${length}" y="${width}" z="${height}">
+                <origin xyz="0.0 0.0 0.0" rpy="0.0 0.0 0.0"/>
+            </xacro:inertial_box>
         </link>
         <joint name="${parent}_to_${prefix}_layer_joint" type="fixed">
             <parent link="${parent}_link"/>
             <child link="${prefix}_layer_link"/>
-            <origin xyz="0 0 ${reflect*0.055}" rpy="0 0 0"/>
+            <xacro:insert_block name="layer_joint_origin"/>
         </joint>
     </xacro:macro>

File: mecabot_body/urdf/chassis/pillar.xacro (robot description, xacro)
@@ -3,11 +3,20 @@
     <xacro:property name="pillar_radius" value="0.002"/>
     <xacro:property name="pillar_length" value="0.055"/>
-    <xacro:property name="pillar_mass" value="0.01"/>
+    <xacro:property name="pillar_mass" value="0.005"/>
     <xacro:property name="pillar_offset_fb" value="0.12"/>
     <xacro:property name="pillar_offset_lr" value="0.055"/>
+    <xacro:macro name="inertial_cylinder" params="mass radius length *origin">
+        <inertial>
+            <xacro:insert_block name="origin"/>
+            <mass value="${mass}" />
+            <inertia ixx="${(1/12) * mass * (3*radius*radius + length*length)}" ixy="0.0" ixz="0.0"
+                    iyy="${(1/12) * mass * (3*radius*radius + length*length)}" iyz="0.0"
+                    izz="${(1/2) * mass * (radius*radius)}" />
+        </inertial>
+    </xacro:macro>
     <xacro:macro name="pillar" params="suffix parent side_FB side_LR">
-        <xacro:macro name="pillar_joint_origin">
+        <xacro:property name="pillar_joint_origin">
             <origin xyz="${pillar_offset_fb*side_FB} ${pillar_offset_lr*side_LR} 0.0" rpy="0.0 0.0 0.0"/>
-        </xacro:macro>
+        </xacro:property>
         <link name="pillar_${suffix}_link">
             <visual>
@@ -26,9 +35,12 @@
                 </geometry>
             </collision>
+            <xacro:inertial_cylinder mass="${pillar_mass}" radius="${pillar_radius}" length="${pillar_length}">
+                <origin xyz="0.0 0.0 ${pillar_length/2}" rpy="0.0 0.0 0.0"/>
+            </xacro:inertial_cylinder>
         </link>
         <joint name="${parent}_to_pillar_${suffix}_joint" type="fixed">
             <parent link="${parent}_link"/>
             <child link="pillar_${suffix}_link"/>
-            <xacro:pillar_joint_origin/>
+            <xacro:insert_block name="pillar_joint_origin"/>
         </joint>
     </xacro:macro>

File: mecabot_body/urdf/mecabot_core.xacro (robot description, xacro)
@@ -11,6 +11,6 @@
     <xacro:property name="wheel_height" value="0.03" />
     <xacro:include filename="$(find mecabot_body)/urdf/includes/materials.xacro"/>
-    <xacro:include filename="$(find mecabot_body)/urdf/parts/pillar.xacro"/>
-    <xacro:include filename="$(find mecabot_body)/urdf/parts/layer.xacro"/>
+    <xacro:include filename="$(find mecabot_body)/urdf/chassis/pillar.xacro"/>
+    <xacro:include filename="$(find mecabot_body)/urdf/chassis/layer.xacro"/>
     <xacro:include filename="$(find mecabot_body)/urdf/wheels/wheel.xacro"/>
     <!-- BASE LINK -->

File: mecabot_body/urdf/wheels/wheel.xacro (robot description, xacro)
@@ -5,16 +5,20 @@
     <xacro:property name="wheel_radius" value="0.03" />
     <xacro:property name="wheel_thickness" value="0.031" />
-    <xacro:property name="wheel_mass" value="0.1" /> <!-- in kg-->
+    <xacro:property name="wheel_mass" value="0.04" /> <!-- in kg-->
     <xacro:property name="wheel_offset_fb" value="0.06215"/>
     <xacro:property name="wheel_offset_lr" value="0.064"/>
-    <xacro:macro name="cylinder_inertia" params="m r h">
-        <inertia  ixx="${m*(3*r*r+h*h)/12}" ixy = "0" ixz = "0"
-                  iyy="${m*r*r/2}" iyz = "0"
-                  izz="${m*(3*r*r+h*h)/12}" />
+    <xacro:macro name="inertial_cylinder" params="mass radius length *origin">
+        <inertial>
+            <xacro:insert_block name="origin"/>
+            <mass value="${mass}" />
+            <inertia ixx="${(1/12) * mass * (3*radius*radius + length*length)}" ixy="0.0" ixz="0.0"
+                    iyy="${(1/12) * mass * (3*radius*radius + length*length)}" iyz="0.0"
+                    izz="${(1/2) * mass * (radius*radius)}" />
+        </inertial>
     </xacro:macro>
     <xacro:macro name="wheel" params="prefix parent side_FB side_LR">
-        <xacro:macro name="wheel_joint_origin">
+        <xacro:property name="wheel_joint_origin">
             <origin xyz="${wheel_offset_fb*side_FB} ${wheel_offset_lr*side_LR} -${motor_offset_z}" rpy="-${PI/2} 0.0 0.0"/>
-        </xacro:macro>
+        </xacro:property>
         <link name="${prefix}_wheel_link">
             <visual name="shaft">
@@ -27,5 +31,5 @@
                 </material>
             </visual>
-            <visual>
+            <visual name="wheel">
                 <origin xyz="0.0 0.0 0.0" rpy="0.0 0.0 0.0"/>
                 <geometry>
@@ -42,17 +46,16 @@
                 </geometry>
             </collision>
-            <inertial>
-                <mass value="${wheel_mass}"/>
-                <xacro:cylinder_inertia  m="${wheel_mass}" r="${wheel_radius}" h="${wheel_thickness}"/>
-            </inertial>
+            <xacro:inertial_cylinder  mass="${wheel_mass}" radius="${wheel_radius}" length="${wheel_thickness}">
+                <origin xyz="0 0 0" rpy="0 0 0"/>
+            </xacro:inertial_cylinder>
         </link>
         <joint name="${prefix}_wheel_joint" type="continuous">
             <parent link="${parent}_link"/>
             <child link="${prefix}_wheel_link"/>
-            <xacro:wheel_joint_origin/>
+            <xacro:insert_block name="wheel_joint_origin" />
             <axis xyz="0 0 1" rpy="0 0 0" />
             <limit effort="100" velocity="100"/>
             <joint_properties damping="0.0" friction="0.0"/>
-          </joint>
+        </joint>
     </xacro:macro>
 </robot>

Commit message: Created a global macro file for physical properties.

File: mecabot_body/urdf/chassis/layer.xacro (robot description, xacro)
@@ -7,5 +7,4 @@
     <xacro:property name="motor_offset_fb" value="0.04"/>
     <xacro:property name="motor_offset_lr" value="0.034"/>
-    <xacro:property name="layer_mass" value="0.07"/>
     <xacro:macro name="base_color">
         <material name="metal">
@@ -27,5 +26,5 @@
         </inertial>
     </xacro:macro>
-    <xacro:macro name="layer" params="prefix parent length width height reflect">
+    <xacro:macro name="layer" params="prefix parent mass length width height reflect">
         <xacro:property name="layer_joint_origin">
             <origin xyz="0 0 ${reflect*0.055}" rpy="0 0 0"/>
@@ -146,5 +145,5 @@
                 </geometry>
             </collision>
-            <xacro:inertial_box mass="${layer_mass}" x="${length}" y="${width}" z="${height}">
+            <xacro:inertial_box mass="${mass}" x="${length}" y="${width}" z="${height}">
                 <origin xyz="0.0 0.0 0.0" rpy="0.0 0.0 0.0"/>
             </xacro:inertial_box>

File: mecabot_body/urdf/chassis/pillar.xacro (robot description, xacro)
@@ -1,7 +1,4 @@
 <?xml version="1.0" encoding="UTF-8"?>
 <robot xmlns:xacro="http://ros.org/wiki/xacro">
-    <xacro:property name="pillar_radius" value="0.002"/>
-    <xacro:property name="pillar_length" value="0.055"/>
-    <xacro:property name="pillar_mass" value="0.005"/>
     <xacro:property name="pillar_offset_fb" value="0.12"/>
     <xacro:property name="pillar_offset_lr" value="0.055"/>
@@ -15,5 +12,5 @@
         </inertial>
     </xacro:macro>
-    <xacro:macro name="pillar" params="suffix parent side_FB side_LR">
+    <xacro:macro name="pillar" params="suffix parent mass radius length side_FB side_LR">
         <xacro:property name="pillar_joint_origin">
             <origin xyz="${pillar_offset_fb*side_FB} ${pillar_offset_lr*side_LR} 0.0" rpy="0.0 0.0 0.0"/>
@@ -21,7 +18,7 @@
         <link name="pillar_${suffix}_link">
             <visual>
-                <origin xyz="0.0 0.0 ${pillar_length/2}" rpy="0.0 0.0 0.0"/>
+                <origin xyz="0.0 0.0 ${length/2}" rpy="0.0 0.0 0.0"/>
                 <geometry>
-                    <cylinder radius="${pillar_radius}" length="${pillar_length}"/>
+                    <cylinder radius="${radius}" length="${length}"/>
                 </geometry>
                 <material name="pillar_color">
@@ -30,11 +27,11 @@
             </visual>
             <collision>
-                <origin xyz="0.0 0.0 ${pillar_length/2}" rpy="0.0 0.0 0.0"/>
+                <origin xyz="0.0 0.0 ${length/2}" rpy="0.0 0.0 0.0"/>
                 <geometry>
-                    <cylinder radius="${pillar_radius}" length="${pillar_length}"/>
+                    <cylinder radius="${radius}" length="${length}"/>
                 </geometry>
             </collision>
-            <xacro:inertial_cylinder mass="${pillar_mass}" radius="${pillar_radius}" length="${pillar_length}">
-                <origin xyz="0.0 0.0 ${pillar_length/2}" rpy="0.0 0.0 0.0"/>
+            <xacro:inertial_cylinder mass="${mass}" radius="${radius}" length="${length}">
+                <origin xyz="0.0 0.0 ${length/2}" rpy="0.0 0.0 0.0"/>
             </xacro:inertial_cylinder>
         </link>

File: mecabot_body/urdf/includes/common_macros.xacro (robot description, xacro)
@@ -1,11 +1,20 @@
 <?xml version="1.0"?>
 <robot xmlns:xacro="http://www.ros.org/wiki/xacro" name="robot_name">
+    <xacro:property name="PI" value="3.1415926535897931" />
+    <!-- Layer and chassis properties -->
     <xacro:property name="layer_l" value="0.255"/>
     <xacro:property name="layer_w" value="0.15"/>
-    <xacro:property name="layer_h" value="0.001"/>
-    <xacro:property name="pillar_radius" value="0.001"/>
-    <xacro:property name="pillar_length" value="0.06"/>
-    <xacro:property name="pillar_mass" value="0.01"/>
-    <xacro:property name="pillar_offset_fr" value="${0.9*layer_l/2}"/>
-    <xacro:property name="pillar_offset_lr" value="${0.9*layer_w/2}"/>
+    <xacro:property name="layer_h" value="0.002"/>
+    <xacro:property name="layer_mass" value="0.07"/>
+    <xacro:property name="chassis_l" value="${layer_l}"/>
+    <xacro:property name="chassis_w" value="${layer_w}"/>
+    <xacro:property name="chassis_h" value="0.07"/>
+    <!-- Wheel properties -->
+    <xacro:property name="wheel_radius" value="0.03" />
+    <xacro:property name="wheel_thickness" value="0.031" />
+    <xacro:property name="wheel_mass" value="0.04" /> <!-- in kg-->
+    <!-- Copper pillar properties -->
+    <xacro:property name="pillar_radius" value="0.002"/>
+    <xacro:property name="pillar_length" value="0.055"/>
+    <xacro:property name="pillar_mass" value="0.005"/>
 </robot>

File: mecabot_body/urdf/mecabot_core.xacro (robot description, xacro)
@@ -1,13 +1,5 @@
 <?xml version="1.0"?>
 <robot xmlns:xacro="http://www.ros.org/wiki/xacro">
-    <xacro:property name="layer_l" value="0.255"/>
-    <xacro:property name="layer_w" value="0.15"/>
-    <xacro:property name="layer_h" value="0.002"/>
-    <xacro:property name="chassis_l" value="${layer_l}"/>
-    <xacro:property name="chassis_w" value="${layer_w}"/>
-    <xacro:property name="chassis_h" value="0.07"/>
-    <xacro:property name="PI" value="3.1415926535897931" />
-    <xacro:property name="wheel_radius" value="0.03" />
-    <xacro:property name="wheel_height" value="0.03" />
+    <xacro:include filename="$(find mecabot_body)/urdf/includes/common_macros.xacro"/>
     <xacro:include filename="$(find mecabot_body)/urdf/includes/materials.xacro"/>
     <xacro:include filename="$(find mecabot_body)/urdf/chassis/pillar.xacro"/>
@@ -24,16 +16,28 @@
     </link>
     <!-- LAYER AND PILLAR LINKS -->
-    <xacro:layer prefix="lower" parent="base" length="${layer_l}" width="${layer_w-wheel_height*2}" height="${layer_h}" reflect="0"/>
-    <xacro:pillar suffix="one" parent="base" side_FB="1" side_LR="0"/>
-    <xacro:pillar suffix="two" parent="base" side_FB="1" side_LR="1"/>
-    <xacro:pillar suffix="three" parent="base" side_FB="1" side_LR="-1"/>
-    <xacro:pillar suffix="four" parent="base" side_FB="-1" side_LR="0"/>
-    <xacro:pillar suffix="five" parent="base" side_FB="-1" side_LR="1"/>
-    <xacro:pillar suffix="six" parent="base" side_FB="-1" side_LR="-1"/>
-    <xacro:layer prefix="upper" parent="base" length="${layer_l}" width="${layer_w-wheel_height*2}" height="${layer_h}" reflect="1"></xacro:layer>
+    <xacro:layer prefix="lower" parent="base" mass="${layer_mass}"
+                length="${layer_l}" width="${layer_w-wheel_thickness*2}" height="${layer_h}" reflect="0"/>
+    <xacro:pillar suffix="one" parent="base" mass="${pillar_mass}"
+                radius="${pillar_radius}" length="${pillar_length}" side_FB="1" side_LR="0"/>
+    <xacro:pillar suffix="two" parent="base" mass="${pillar_mass}"
+                radius="${pillar_radius}" length="${pillar_length}" side_FB="1" side_LR="1"/>
+    <xacro:pillar suffix="three" parent="base" mass="${pillar_mass}"
+                 radius="${pillar_radius}" length="${pillar_length}" side_FB="1" side_LR="-1"/>
+    <xacro:pillar suffix="four" parent="base" mass="${pillar_mass}"
+                radius="${pillar_radius}" length="${pillar_length}" side_FB="-1" side_LR="0"/>
+    <xacro:pillar suffix="five" parent="base" mass="${pillar_mass}"
+                radius="${pillar_radius}" length="${pillar_length}" side_FB="-1" side_LR="1"/>
+    <xacro:pillar suffix="six" parent="base" mass="${pillar_mass}"
+                radius="${pillar_radius}" length="${pillar_length}" side_FB="-1" side_LR="-1"/>
+    <xacro:layer prefix="upper" parent="base" mass="${layer_mass}"
+                length="${layer_l}" width="${layer_w-wheel_thickness*2}" height="${layer_h}" reflect="1"/>
     <!-- MECANUM WHEEL LINKS -->
-    <xacro:wheel prefix="front_left" parent="base" side_FB="1" side_LR="1"/>
-    <xacro:wheel prefix="front_right" parent="base" side_FB="1" side_LR="-1"/>
-    <xacro:wheel prefix="back_left" parent="base" side_FB="-1" side_LR="1"/>
-    <xacro:wheel prefix="back_right" parent="base" side_FB="-1" side_LR="-1"/>
+    <xacro:wheel prefix="front_left" parent="base" mass="${wheel_mass}"
+                radius="${wheel_radius}" thickness="${wheel_thickness}" side_FB="1" side_LR="1"/>
+    <xacro:wheel prefix="front_right" parent="base" mass="${wheel_mass}"
+                radius="${wheel_radius}" thickness="${wheel_thickness}" side_FB="1" side_LR="-1"/>
+    <xacro:wheel prefix="back_left" parent="base" mass="${wheel_mass}"
+                radius="${wheel_radius}" thickness="${wheel_thickness}" side_FB="-1" side_LR="1"/>
+    <xacro:wheel prefix="back_right" parent="base" mass="${wheel_mass}"
+                radius="${wheel_radius}" thickness="${wheel_thickness}" side_FB="-1" side_LR="-1"/>
 </robot>

File: mecabot_body/urdf/wheels/wheel.xacro (robot description, xacro)
@@ -1,9 +1,6 @@
 <?xml version="1.0"?>
 <robot xmlns:xacro="http://www.ros.org/wiki/xacro">
-    <xacro:property name="motor_offset_z" value="0.009" />
     <xacro:property name="PI" value="3.1415926535897931" />
-    <xacro:property name="wheel_radius" value="0.03" />
-    <xacro:property name="wheel_thickness" value="0.031" />
-    <xacro:property name="wheel_mass" value="0.04" /> <!-- in kg-->
+    <xacro:property name="wheel_offset_z" value="0.009" />
     <xacro:property name="wheel_offset_fb" value="0.06215"/>
     <xacro:property name="wheel_offset_lr" value="0.064"/>
@@ -17,11 +14,11 @@
         </inertial>
     </xacro:macro>
-    <xacro:macro name="wheel" params="prefix parent side_FB side_LR">
+    <xacro:macro name="wheel" params="prefix parent mass radius thickness side_FB side_LR">
         <xacro:property name="wheel_joint_origin">
-            <origin xyz="${wheel_offset_fb*side_FB} ${wheel_offset_lr*side_LR} -${motor_offset_z}" rpy="-${PI/2} 0.0 0.0"/>
+            <origin xyz="${wheel_offset_fb*side_FB} ${wheel_offset_lr*side_LR} -${wheel_offset_z}" rpy="-${PI/2} 0.0 0.0"/>
         </xacro:property>
         <link name="${prefix}_wheel_link">
             <visual name="shaft">
-                <origin xyz="0.0 0.0 ${-1 * side_LR * wheel_thickness/2}"/>
+                <origin xyz="0.0 0.0 ${-1 * side_LR * thickness/2}"/>
                 <geometry>
                     <cylinder radius="0.0025" length="0.02"/>
@@ -34,5 +31,5 @@
                 <origin xyz="0.0 0.0 0.0" rpy="0.0 0.0 0.0"/>
                 <geometry>
-                    <cylinder radius="${wheel_radius}" length="${wheel_thickness}"/>
+                    <cylinder radius="${radius}" length="${thickness}"/>
                 </geometry>
                 <material name="yellow">
@@ -43,8 +40,8 @@
                 <origin xyz="0 0 0" rpy="0 0 0" />
                 <geometry>
-                    <cylinder radius="${wheel_radius}" length="${wheel_thickness}"/>
+                    <cylinder radius="${radius}" length="${thickness}"/>
                 </geometry>
             </collision>
-            <xacro:inertial_cylinder  mass="${wheel_mass}" radius="${wheel_radius}" length="${wheel_thickness}">
+            <xacro:inertial_cylinder  mass="${mass}" radius="${radius}" length="${thickness}">
                 <origin xyz="0 0 0" rpy="0 0 0"/>
             </xacro:inertial_cylinder>
