Commit message: Added gazebo simulation

File: mecabot_body/urdf/chassis/layer.xacro (robot description, xacro)
@@ -8,6 +8,6 @@
     <xacro:property name="motor_offset_lr" value="0.034"/>
     <xacro:macro name="base_color">
-        <material name="metal">
-            <color rgba="0.5 0.5 0.5 1.0"/>
+        <material name="blue">
+            <color rgba="0.0 0.2 1.0 1.0"/>
         </material>
     </xacro:macro>
@@ -97,5 +97,6 @@
                 </visual>
             </xacro:if>
-            <visual name="${prefix}_top_left_piece">
+            <!-- Top left piece -->
+            <visual>
                 <origin xyz="${length/2-side_piece_size/2} ${width/2+side_piece_size/2} 0" rpy="0.0 0.0 0.0"/>
                 <geometry>
@@ -104,5 +105,6 @@
                 <xacro:base_color/>
             </visual>
-            <visual name="${prefix}_top_right_piece">
+            <!-- Top right piece -->
+            <visual>
                 <origin xyz="${length/2-side_piece_size/2} -${width/2+side_piece_size/2} 0" rpy="0.0 0.0 0.0"/>
                 <geometry>
@@ -111,5 +113,6 @@
                 <xacro:base_color/>
             </visual>
-            <visual name="${prefix}_mid_left_piece">
+            <!-- Middle left piece -->
+            <visual>
                 <origin xyz="0.0 ${width/2+side_piece_size/2} 0" rpy="0.0 0.0 0.0"/>
                 <geometry>
@@ -118,5 +121,6 @@
                 <xacro:base_color/>
             </visual>
-            <visual name="${prefix}_mid_right_piece">
+            <!-- Middle right piece -->
+            <visual>
                 <origin xyz="0.0 -${width/2+side_piece_size/2} 0" rpy="0.0 0.0 0.0"/>
                 <geometry>
@@ -125,5 +129,6 @@
                 <xacro:base_color/>
             </visual>
-            <visual name="${prefix}_bot_left_piece">
+            <!-- Bottom left piece -->
+            <visual>
                 <origin xyz="-${length/2-side_piece_size/2} ${width/2+side_piece_size/2} 0" rpy="0.0 0.0 0.0"/>
                 <geometry>
@@ -132,5 +137,6 @@
                 <xacro:base_color/>
             </visual>
-            <visual name="${prefix}_bot_right_piece">
+            <!-- Bottom right piece -->
+            <visual>
                 <origin xyz="-${length/2-side_piece_size/2} -${width/2+side_piece_size/2} 0" rpy="0.0 0.0 0.0"/>
                 <geometry>
@@ -154,4 +160,18 @@
             <xacro:insert_block name="layer_joint_origin"/>
         </joint>
+        <gazebo reference="${prefix}_layer_link">
+            <material>Gazebo/Blue</material>
+            <visual name="direction_piece_1">
+                <material>
+                    <diffuse>0 0 0 1</diffuse>
+                </material>
+            </visual>
+            <visual name="direction_piece_2">
+                <material>Gazebo/Red</material>
+            </visual>
+            <visual name="direction_piece_3">
+                <material>Gazebo/Red</material>
+            </visual>
+        </gazebo>
     </xacro:macro>
 </robot>

File: mecabot_body/urdf/chassis/pillar.xacro (robot description, xacro)
@@ -41,4 +41,7 @@
             <xacro:insert_block name="pillar_joint_origin"/>
         </joint>
+        <gazebo reference="pillar_${suffix}_link">
+            <material>Gazebo/Orange</material>
+        </gazebo>
     </xacro:macro>
 </robot>

File: mecabot_body/urdf/wheels/wheel.xacro (robot description, xacro)
@@ -28,5 +28,5 @@
                 </material>
             </visual>
-            <visual name="wheel">
+            <visual>
                 <origin xyz="0.0 0.0 0.0" rpy="0.0 0.0 0.0"/>
                 <geometry>
@@ -55,4 +55,12 @@
             <joint_properties damping="0.0" friction="0.0"/>
         </joint>
+        <gazebo reference="${prefix}_wheel_link">
+            <material>Gazebo/Yellow</material>
+            <visual name="direction_piece_1">
+                <material>
+                    <diffuse>0 0 0 1</diffuse>
+                </material>
+            </visual>
+        </gazebo>
     </xacro:macro>
 </robot>

Commit message: Added visual change in Gazebo

File: mecabot_body/urdf/chassis/layer.xacro (robot description, xacro)
@@ -38,33 +38,4 @@
                 <xacro:base_color/>
             </visual>
-            <xacro:if value="${prefix == 'upper'}">
-                <visual name="direction_piece_1">
-                    <origin xyz="${length/2-side_piece_size/2} 0.0 ${height/2}" rpy="0.0 0.0 0.0"/>
-                    <geometry>
-                        <box size="${side_piece_size} ${side_piece_size} ${height/2}"/>
-                    </geometry>
-                    <material name="header">
-                        <color rgba="1.0 0.0 0.0 1.0"/>
-                    </material>
-                </visual>
-                <visual name="direction_piece_2">
-                    <origin xyz="${length/2-1.5*side_piece_size} ${width/2-side_piece_size/2} ${height/2}" rpy="0.0 0.0 0.0"/>
-                    <geometry>
-                        <box size="${side_piece_size} ${side_piece_size} ${height/2}"/>
-                    </geometry>
-                    <material name="header">
-                        <color rgba="1.0 0.0 0.0 1.0"/>
-                    </material>
-                </visual>
-                <visual name="direction_piece_3">
-                    <origin xyz="${length/2-1.5*side_piece_size} -${width/2-side_piece_size/2} ${height/2}" rpy="0.0 0.0 0.0"/>
-                    <geometry>
-                        <box size="${side_piece_size} ${side_piece_size} ${height}"/>
-                    </geometry>
-                    <material name="header">
-                        <color rgba="1.0 0.0 0.0 1.0"/>
-                    </material>
-                </visual>
-            </xacro:if>
             <xacro:if value="${prefix == 'lower'}">
                 <visual name="FL_motor">
@@ -162,16 +133,64 @@
         <gazebo reference="${prefix}_layer_link">
             <material>Gazebo/Blue</material>
-            <visual name="direction_piece_1">
-                <material>
-                    <diffuse>0 0 0 1</diffuse>
+        </gazebo>
+        <xacro:if value="${prefix == 'upper'}">
+        <link name="direction_piece_1">
+            <visual>
+                <origin xyz="0 0 0" rpy="0.0 0.0 0.0"/>
+                <geometry>
+                    <box size="${side_piece_size} ${side_piece_size} ${height/2}"/>
+                </geometry>
+                <material name="header">
+                    <color rgba="1.0 0.0 0.0 1.0"/>
                 </material>
             </visual>
-            <visual name="direction_piece_2">
-                <material>Gazebo/Red</material>
+        </link>
+        <joint name="direction_piece_1_joint" type="fixed">
+            <origin xyz="${length/2-side_piece_size/2} 0.0 ${height/2}" rpy="0.0 0.0 0.0"/>
+            <parent link="${prefix}_layer_link"/>
+            <child link="direction_piece_1"/>
+        </joint>
+        <gazebo reference="direction_piece_1">
+            <material>Gazebo/Red</material>
+        </gazebo>
+        <link name="direction_piece_2">
+            <visual>
+                <origin xyz="0 0 0" rpy="0.0 0.0 0.0"/>
+                <geometry>
+                    <box size="${side_piece_size} ${side_piece_size} ${height/2}"/>
+                </geometry>
+                <material name="header">
+                    <color rgba="1.0 0.0 0.0 1.0"/>
+                </material>
             </visual>
-            <visual name="direction_piece_3">
-                <material>Gazebo/Red</material>
+        </link>
+        <joint name="direction_piece_2_joint" type="fixed">
+            <origin xyz="${length/2-1.5*side_piece_size} ${width/2-side_piece_size/2} ${height/2}" rpy="0.0 0.0 0.0"/>
+            <parent link="${prefix}_layer_link"/>
+            <child link="direction_piece_2"/>
+        </joint>
+        <gazebo reference="direction_piece_2">
+            <material>Gazebo/Red</material>
+        </gazebo>
+        <link name="direction_piece_3">
+            <visual>
+                <origin xyz="0 0 0" rpy="0.0 0.0 0.0"/>
+                <geometry>
+                    <box size="${side_piece_size} ${side_piece_size} ${height}"/>
+                </geometry>
+                <material name="header">
+                    <color rgba="1.0 0.0 0.0 1.0"/>
+                </material>
             </visual>
+        </link>
+        <joint name="direction_piece_3_joint" type="fixed">
+            <origin xyz="${length/2-1.5*side_piece_size} -${width/2-side_piece_size/2} ${height/2}" rpy="0.0 0.0 0.0"/>
+            <parent link="${prefix}_layer_link"/>
+            <child link="direction_piece_3"/>
+        </joint>
+        <gazebo reference="direction_piece_3">
+            <material>Gazebo/Red</material>
         </gazebo>
+    </xacro:if>
     </xacro:macro>
 </robot>

Commit message: Added visual for mecanum wheel & changed motor visual definition

File: mecabot_body/urdf/chassis/layer.xacro (robot description, xacro)
@@ -7,13 +7,34 @@
     <xacro:property name="motor_offset_fb" value="0.04"/>
     <xacro:property name="motor_offset_lr" value="0.034"/>
-    <xacro:macro name="base_color">
+    <xacro:property name="shaft_radius" value="0.0025"/>
+    <xacro:property name="shaft_length" value="0.02"/>
+    <xacro:property name="shaft_offset_fb" value="0.06215"/>
+    <xacro:property name="base_material">
         <material name="blue">
             <color rgba="0.0 0.2 1.0 1.0"/>
         </material>
-    </xacro:macro>
-    <xacro:macro name="motor_color">
-        <material name="motor">
+    </xacro:property>
+    <xacro:property name="motor_material">
+        <material name="motor_yellow">
             <color rgba="${247/255} ${200/255} ${60/255} 1.0"/>
         </material>
+    </xacro:property>
+    <xacro:macro name="motor_visual" params="name side_FB side_LR">
+        <visual name="${name}">
+            <origin xyz="${motor_offset_fb*side_FB} ${motor_offset_lr*side_LR} -${motor_h/2}" rpy="0.0 0.0 0.0"/>
+            <geometry>
+                <box size="${motor_l} ${motor_w} ${motor_h}"/>
+            </geometry>
+            <xacro:insert_block name="motor_material"/>
+        </visual>
+        <visual name="${name}_shaft">
+            <origin xyz="${shaft_offset_fb*side_FB} ${(motor_offset_lr + shaft_length)*side_LR} -${motor_h/2}" rpy="-${PI/2} 0.0 0.0"/>
+            <geometry>
+                <cylinder radius="${shaft_radius}" length="${shaft_length}"/>
+            </geometry>
+            <material name="white">
+                <color rgba="1.0 1.0 1.0 1.0"/>
+            </material>
+        </visual>
     </xacro:macro>
     <xacro:macro name="inertial_box" params="mass x y z *origin">
@@ -36,35 +57,11 @@
                     <box size="${length} ${width} ${height}"/>
                 </geometry>
-                <xacro:base_color/>
+                <xacro:insert_block name="base_material"/>
             </visual>
             <xacro:if value="${prefix == 'lower'}">
-                <visual name="FL_motor">
-                    <origin xyz="${motor_offset_fb} ${motor_offset_lr} -${motor_h/2}" rpy="0.0 0.0 0.0"/>
-                    <geometry>
-                        <box size="${motor_l} ${motor_w} ${motor_h}"/>
-                    </geometry>
-                    <xacro:motor_color/>
-                </visual>
-                <visual name="FR_motor">
-                    <origin xyz="${motor_offset_fb} -${motor_offset_lr} -${motor_h/2}" rpy="0.0 0.0 0.0"/>
-                    <geometry>
-                        <box size="${motor_l} ${motor_w} ${motor_h}"/>
-                    </geometry>
-                    <xacro:motor_color/>
-                </visual>
-                <visual name="BL_motor">
-                    <origin xyz="-${motor_offset_fb} ${motor_offset_lr} -${motor_h/2}" rpy="0.0 0.0 0.0"/>
-                    <geometry>
-                        <box size="${motor_l} ${motor_w} ${motor_h}"/>
-                    </geometry>
-                    <xacro:motor_color/>
-                </visual>
-                <visual name="BR_motor">
-                    <origin xyz="-${motor_offset_fb} -${motor_offset_lr} -${motor_h/2}" rpy="0.0 0.0 0.0"/>
-                    <geometry>
-                        <box size="${motor_l} ${motor_w} ${motor_h}"/>
-                    </geometry>
-                    <xacro:motor_color/>
-                </visual>
+                <xacro:motor_visual name="FL_motor" side_FB="1" side_LR="1"/>
+                <xacro:motor_visual name="FR_motor" side_FB="1" side_LR="-1"/>
+                <xacro:motor_visual name="BL_motor" side_FB="-1" side_LR="1"/>
+                <xacro:motor_visual name="BR_motor" side_FB="-1" side_LR="-1"/>
             </xacro:if>
             <!-- Top left piece -->
@@ -74,5 +71,5 @@
                     <box size="${side_piece_size} ${side_piece_size} ${height}"/>
                 </geometry>
-                <xacro:base_color/>
+                <xacro:insert_block name="base_material"/>
             </visual>
             <!-- Top right piece -->
@@ -82,5 +79,5 @@
                     <box size="${side_piece_size} ${side_piece_size} ${height}"/>
                 </geometry>
-                <xacro:base_color/>
+                <xacro:insert_block name="base_material"/>
             </visual>
             <!-- Middle left piece -->
@@ -90,5 +87,5 @@
                     <box size="${side_piece_size*1.8} ${side_piece_size} ${height}"/>
                 </geometry>
-                <xacro:base_color/>
+                <xacro:insert_block name="base_material"/>
             </visual>
             <!-- Middle right piece -->
@@ -98,5 +95,5 @@
                     <box size="${side_piece_size*1.8} ${side_piece_size} ${height}"/>
                 </geometry>
-                <xacro:base_color/>
+                <xacro:insert_block name="base_material"/>
             </visual>
             <!-- Bottom left piece -->
@@ -106,5 +103,5 @@
                     <box size="${side_piece_size} ${side_piece_size} ${height}"/>
                 </geometry>
-                <xacro:base_color/>
+                <xacro:insert_block name="base_material"/>
             </visual>
             <!-- Bottom right piece -->
@@ -114,5 +111,5 @@
                     <box size="${side_piece_size} ${side_piece_size} ${height}"/>
                 </geometry>
-                <xacro:base_color/>
+                <xacro:insert_block name="base_material"/>
             </visual>
             <collision>

File: mecabot_body/urdf/mecabot_core.xacro (robot description, xacro)
@@ -6,4 +6,5 @@
     <xacro:include filename="$(find mecabot_body)/urdf/chassis/layer.xacro"/>
     <xacro:include filename="$(find mecabot_body)/urdf/wheels/wheel.xacro"/>
+    <xacro:include filename="$(find mecabot_body)/urdf/wheels/mecanum_wheel.xacro"/>
     <!-- BASE LINK -->
     <link name="base_link">
@@ -33,11 +34,11 @@
                 length="${layer_l}" width="${layer_w-wheel_thickness*2}" height="${layer_h}" reflect="1"/>
     <!-- MECANUM WHEEL LINKS -->
-    <xacro:wheel prefix="front_left" parent="base" mass="${wheel_mass}"
+    <xacro:mecanum_wheel prefix="front_left" parent="base" mass="${wheel_mass}"
                 radius="${wheel_radius}" thickness="${wheel_thickness}" side_FB="1" side_LR="1"/>
-    <xacro:wheel prefix="front_right" parent="base" mass="${wheel_mass}"
+    <xacro:mecanum_wheel prefix="front_right" parent="base" mass="${wheel_mass}"
                 radius="${wheel_radius}" thickness="${wheel_thickness}" side_FB="1" side_LR="-1"/>
-    <xacro:wheel prefix="back_left" parent="base" mass="${wheel_mass}"
+    <xacro:mecanum_wheel prefix="back_left" parent="base" mass="${wheel_mass}"
                 radius="${wheel_radius}" thickness="${wheel_thickness}" side_FB="-1" side_LR="1"/>
-    <xacro:wheel prefix="back_right" parent="base" mass="${wheel_mass}"
+    <xacro:mecanum_wheel prefix="back_right" parent="base" mass="${wheel_mass}"
                 radius="${wheel_radius}" thickness="${wheel_thickness}" side_FB="-1" side_LR="-1"/>
 </robot>

File: mecabot_body/urdf/wheels/wheel.xacro (robot description, xacro)
@@ -52,14 +52,8 @@
             <xacro:insert_block name="wheel_joint_origin" />
             <axis xyz="0 0 1" rpy="0 0 0" />
-            <limit effort="100" velocity="100"/>
-            <joint_properties damping="0.0" friction="0.0"/>
+            <dynamic damping="0.01" friction="0.0"/>
         </joint>
         <gazebo reference="${prefix}_wheel_link">
             <material>Gazebo/Yellow</material>
-            <visual name="direction_piece_1">
-                <material>
-                    <diffuse>0 0 0 1</diffuse>
-                </material>
-            </visual>
         </gazebo>
     </xacro:macro>
