Commit message: Updated LiDAR simulation & Improved Xacro files

File: mecabot_body/urdf/chassis/layer.xacro (robot description, xacro)
@@ -1,13 +1,4 @@
 <?xml version="1.0"?>
 <robot xmlns:xacro="http://www.ros.org/wiki/xacro">
-    <xacro:property name="side_piece_size" value="0.03"/>
-    <xacro:property name="motor_l" value="0.07"/>
-    <xacro:property name="motor_w" value="0.022"/>
-    <xacro:property name="motor_h" value="0.018"/>
-    <xacro:property name="motor_offset_fb" value="0.04"/>
-    <xacro:property name="motor_offset_lr" value="0.034"/>
-    <xacro:property name="shaft_radius" value="0.0025"/>
-    <xacro:property name="shaft_length" value="0.02"/>
-    <xacro:property name="shaft_offset_fb" value="0.06215"/>
     <xacro:property name="base_material">
         <material name="blue">
@@ -38,18 +29,9 @@
         </visual>
     </xacro:macro>
-    <xacro:macro name="inertial_box" params="mass x y z *origin">
-        <inertial>
-            <xacro:insert_block name="origin"/>
-            <mass value="${mass}" />
-            <inertia ixx="${(1/12) * mass * (y*y+z*z)}" ixy="0.0" ixz="0.0"
-                    iyy="${(1/12) * mass * (x*x+z*z)}" iyz="0.0"
-                    izz="${(1/12) * mass * (x*x+y*y)}" />
-        </inertial>
-    </xacro:macro>
     <xacro:macro name="layer" params="prefix parent mass length width height reflect">
         <xacro:property name="layer_joint_origin">
             <origin xyz="0 0 ${reflect*0.055}" rpy="0 0 0"/>
         </xacro:property>
-        <link name="${prefix}_layer_link">
+        <link name="${prefix}_link">
             <visual>
                 <origin xyz="0 0 0" rpy="0 0 0"/>
@@ -59,5 +41,5 @@
                 <xacro:insert_block name="base_material"/>
             </visual>
-            <xacro:if value="${prefix == 'lower'}">
+            <xacro:if value="${prefix == 'lower_layer'}">
                 <xacro:motor_visual name="FL_motor" side_FB="1" side_LR="1"/>
                 <xacro:motor_visual name="FR_motor" side_FB="1" side_LR="-1"/>
@@ -65,5 +47,5 @@
                 <xacro:motor_visual name="BR_motor" side_FB="-1" side_LR="-1"/>
             </xacro:if>
-            <!-- Top left piece -->
+            <!-- Front left piece -->
             <visual>
                 <origin xyz="${length/2-side_piece_size/2} ${width/2+side_piece_size/2} 0" rpy="0.0 0.0 0.0"/>
@@ -73,5 +55,5 @@
                 <xacro:insert_block name="base_material"/>
             </visual>
-            <!-- Top right piece -->
+            <!-- Front right piece -->
             <visual>
                 <origin xyz="${length/2-side_piece_size/2} -${width/2+side_piece_size/2} 0" rpy="0.0 0.0 0.0"/>
@@ -97,5 +79,5 @@
                 <xacro:insert_block name="base_material"/>
             </visual>
-            <!-- Bottom left piece -->
+            <!-- Back left piece -->
             <visual>
                 <origin xyz="-${length/2-side_piece_size/2} ${width/2+side_piece_size/2} 0" rpy="0.0 0.0 0.0"/>
@@ -105,5 +87,5 @@
                 <xacro:insert_block name="base_material"/>
             </visual>
-            <!-- Bottom right piece -->
+            <!-- Back right piece -->
             <visual>
                 <origin xyz="-${length/2-side_piece_size/2} -${width/2+side_piece_size/2} 0" rpy="0.0 0.0 0.0"/>
@@ -123,13 +105,13 @@
             </xacro:inertial_box>
         </link>
-        <joint name="${parent}_to_${prefix}_layer_joint" type="fixed">
+        <joint name="${parent}_to_${prefix}_joint" type="fixed">
             <parent link="${parent}_link"/>
-            <child link="${prefix}_layer_link"/>
+            <child link="${prefix}_link"/>
             <xacro:insert_block name="layer_joint_origin"/>
         </joint>
-        <gazebo reference="${prefix}_layer_link">
+        <gazebo reference="${prefix}_link">
             <material>Gazebo/Blue</material>
         </gazebo>
-        <xacro:if value="${prefix == 'upper'}">
+        <xacro:if value="${prefix == 'upper_layer'}">
         <link name="direction_piece_1">
             <visual>
@@ -145,5 +127,5 @@
         <joint name="direction_piece_1_joint" type="fixed">
             <origin xyz="${length/2-side_piece_size/2} 0.0 ${height/2}" rpy="0.0 0.0 0.0"/>
-            <parent link="${prefix}_layer_link"/>
+            <parent link="${prefix}_link"/>
             <child link="direction_piece_1"/>
         </joint>
@@ -164,5 +146,5 @@
         <joint name="direction_piece_2_joint" type="fixed">
             <origin xyz="${length/2-1.5*side_piece_size} ${width/2-side_piece_size/2} ${height/2}" rpy="0.0 0.0 0.0"/>
-            <parent link="${prefix}_layer_link"/>
+            <parent link="${prefix}_link"/>
             <child link="direction_piece_2"/>
         </joint>
@@ -183,5 +165,5 @@
         <joint name="direction_piece_3_joint" type="fixed">
             <origin xyz="${length/2-1.5*side_piece_size} -${width/2-side_piece_size/2} ${height/2}" rpy="0.0 0.0 0.0"/>
-            <parent link="${prefix}_layer_link"/>
+            <parent link="${prefix}_link"/>
             <child link="direction_piece_3"/>
         </joint>

File: mecabot_body/urdf/chassis/pillar.xacro (robot description, xacro)
@@ -1,15 +1,4 @@
 <?xml version="1.0" encoding="UTF-8"?>
 <robot xmlns:xacro="http://ros.org/wiki/xacro">
-    <xacro:property name="pillar_offset_fb" value="0.12"/>
-    <xacro:property name="pillar_offset_lr" value="0.055"/>
-    <xacro:macro name="inertial_cylinder" params="mass radius length *origin">
-        <inertial>
-            <xacro:insert_block name="origin"/>
-            <mass value="${mass}" />
-            <inertia ixx="${(1/12) * mass * (3*radius*radius + length*length)}" ixy="0.0" ixz="0.0"
-                    iyy="${(1/12) * mass * (3*radius*radius + length*length)}" iyz="0.0"
-                    izz="${(1/2) * mass * (radius*radius)}" />
-        </inertial>
-    </xacro:macro>
     <xacro:macro name="pillar" params="suffix parent mass radius length side_FB side_LR">
         <xacro:property name="pillar_joint_origin">

File: mecabot_body/urdf/includes/common_macros.xacro (robot description, xacro)
@@ -2,4 +2,23 @@
 <robot xmlns:xacro="http://www.ros.org/wiki/xacro" name="robot_name">
     <xacro:property name="PI" value="3.1415926535897931" />
+    <!-- Basic shapes' inertia -->
+    <xacro:macro name="inertial_cylinder" params="mass radius length *origin">
+        <inertial>
+            <xacro:insert_block name="origin"/>
+            <mass value="${mass}" />
+            <inertia ixx="${(1/12) * mass * (3*radius*radius + length*length)}" ixy="0.0" ixz="0.0"
+                    iyy="${(1/12) * mass * (3*radius*radius + length*length)}" iyz="0.0"
+                    izz="${(1/2) * mass * (radius*radius)}" />
+        </inertial>
+    </xacro:macro>
+    <xacro:macro name="inertial_box" params="mass x y z *origin">
+        <inertial>
+            <xacro:insert_block name="origin"/>
+            <mass value="${mass}" />
+            <inertia ixx="${(1/12) * mass * (y*y+z*z)}" ixy="0.0" ixz="0.0"
+                    iyy="${(1/12) * mass * (x*x+z*z)}" iyz="0.0"
+                    izz="${(1/12) * mass * (x*x+y*y)}" />
+        </inertial>
+    </xacro:macro>
     <!-- Layer and chassis properties -->
     <xacro:property name="layer_l" value="0.255"/>
@@ -7,4 +26,13 @@
     <xacro:property name="layer_h" value="0.002"/>
     <xacro:property name="layer_mass" value="0.07"/>
+    <xacro:property name="side_piece_size" value="0.03"/>
+    <xacro:property name="motor_l" value="0.07"/>
+    <xacro:property name="motor_w" value="0.022"/>
+    <xacro:property name="motor_h" value="0.018"/>
+    <xacro:property name="motor_offset_fb" value="0.04"/>
+    <xacro:property name="motor_offset_lr" value="0.034"/>
+    <xacro:property name="shaft_radius" value="0.0025"/>
+    <xacro:property name="shaft_length" value="0.02"/>
+    <xacro:property name="shaft_offset_fb" value="0.06215"/>
     <xacro:property name="chassis_l" value="${layer_l}"/>
     <xacro:property name="chassis_w" value="${layer_w}"/>
@@ -14,7 +42,16 @@
     <xacro:property name="wheel_thickness" value="0.031" />
     <xacro:property name="wheel_mass" value="0.04" /> <!-- in kg-->
+    <xacro:property name="wheel_offset_z" value="0.009" />
+    <xacro:property name="wheel_offset_fb" value="0.06215"/>
+    <xacro:property name="wheel_offset_lr" value="0.064"/>
     <!-- Copper pillar properties -->
     <xacro:property name="pillar_radius" value="0.002"/>
     <xacro:property name="pillar_length" value="0.055"/>
     <xacro:property name="pillar_mass" value="0.005"/>
+    <xacro:property name="pillar_offset_fb" value="0.12"/>
+    <xacro:property name="pillar_offset_lr" value="0.055"/>
+    <!-- LiDAR properties -->
+    <xacro:property name="lidar_radius" value="0.035"/>
+    <xacro:property name="lidar_height" value="0.03"/>
+    <xacro:property name="lidar_mass" value="0.29"/>
 </robot>

File: mecabot_body/urdf/mecabot_core.xacro (robot description, xacro)
@@ -7,4 +7,6 @@
     <xacro:include filename="$(find mecabot_body)/urdf/wheels/wheel.xacro"/>
     <xacro:include filename="$(find mecabot_body)/urdf/wheels/mecanum_wheel.xacro"/>
+    <xacro:include filename="$(find mecabot_body)/urdf/sensors/lidar.xacro"/>
+    <xacro:include filename="$(find mecabot_body)/urdf/mecabot.gazebo.xacro"/>
     <!-- BASE LINK -->
     <link name="base_link">
@@ -17,5 +19,5 @@
     </link>
     <!-- LAYER AND PILLAR LINKS -->
-    <xacro:layer prefix="lower" parent="base" mass="${layer_mass}"
+    <xacro:layer prefix="lower_layer" parent="base" mass="${layer_mass}"
                 length="${layer_l}" width="${layer_w-wheel_thickness*2}" height="${layer_h}" reflect="0"/>
     <xacro:pillar suffix="one" parent="base" mass="${pillar_mass}"
@@ -31,5 +33,5 @@
     <xacro:pillar suffix="six" parent="base" mass="${pillar_mass}"
                 radius="${pillar_radius}" length="${pillar_length}" side_FB="-1" side_LR="-1"/>
-    <xacro:layer prefix="upper" parent="base" mass="${layer_mass}"
+    <xacro:layer prefix="upper_layer" parent="base" mass="${layer_mass}"
                 length="${layer_l}" width="${layer_w-wheel_thickness*2}" height="${layer_h}" reflect="1"/>
     <!-- MECANUM WHEEL LINKS -->
@@ -42,3 +44,11 @@
     <xacro:mecanum_wheel prefix="back_right" parent="base" mass="${wheel_mass}"
                 radius="${wheel_radius}" thickness="${wheel_thickness}" side_FB="-1" side_LR="-1"/>
+    <!-- LIDAR -->
+    <xacro:lidar parent="upper_layer"/>
+    <gazebo>
+        <plugin name="joint_state_publisher" filename="libgazebo_ros_joint_state_publisher.so">
+            <jointName>front_left_wheel_joint, front_right_wheel_joint, back_left_wheel_joint, back_right_wheel_joint</jointName>
+        </plugin>
+    </gazebo>
+    <xacro:mecanum_drive/>
 </robot>

File: mecabot_body/urdf/wheels/mecanum_wheel.xacro (robot description, xacro)
@@ -1,17 +1,4 @@
 <?xml version="1.0"?>
 <robot xmlns:xacro="http://www.ros.org/wiki/xacro">
-    <xacro:property name="PI" value="3.1415926535897931" />
-    <xacro:property name="wheel_offset_z" value="0.009" />
-    <xacro:property name="wheel_offset_fb" value="0.06215"/>
-    <xacro:property name="wheel_offset_lr" value="0.064"/>
-    <xacro:macro name="inertial_cylinder" params="mass radius length *origin">
-        <inertial>
-            <xacro:insert_block name="origin"/>
-            <mass value="${mass}" />
-            <inertia ixx="${(1/12) * mass * (3*radius*radius + length*length)}" ixy="0.0" ixz="0.0"
-                    iyy="${(1/12) * mass * (3*radius*radius + length*length)}" iyz="0.0"
-                    izz="${(1/2) * mass * (radius*radius)}" />
-        </inertial>
-    </xacro:macro>
     <xacro:macro name="mecanum_wheel" params="prefix parent mass radius thickness side_FB side_LR">
         <xacro:property name="wheel_joint_origin">
@@ -64,5 +51,8 @@
         </joint>
         <gazebo reference="${prefix}_wheel_link">
-            <material>Gazebo/Yellow</material>
+            <material>Gazebo/Grey</material>
+            <mu1>0.0</mu1>
+            <mu2>0.0</mu2>
+            <TurnGravityOff>false</TurnGravityOff>
         </gazebo>
     </xacro:macro>
